Commit message: effort and path

File: powerarm_ws_gazebo/src/powerarm_urdf/urdf/powerarm_urdf.urdf (robot description, URDF)
Before this commit: robot powerarm_urdf, 7 links, 6 joints
Joints:
- joint elbow_joint: limit lower=0 upper=1.5708 effort=0 velocity=1.2 -> lower=0 upper=1.5708 effort=200 velocity=1.2
- joint shoulder_joint_1: limit lower=-1.5708 upper=0.785398 effort=0 velocity=1.2 -> lower=-1.5708 upper=0.785398 effort=200 velocity=1.2
- joint shoulder_joint_2: limit lower=-0.5236 upper=1.5708 effort=0 velocity=1.2 -> lower=-0.5236 upper=1.5708 effort=200 velocity=1.2
- joint shoulder_joint_3: limit lower=-1.5708 upper=1.5708 effort=0 velocity=1.2 -> lower=-1.5708 upper=1.5708 effort=200 velocity=1.2
